Commit message: CBF測試

File: openarm_urdf/openarm_bimanual.urdf (robot description, URDF)
Before this commit: robot openarm, 26 links, 25 joints
Links:
- link openarm_left_hand_tcp: mass None -> 1e-05
- link openarm_right_hand_tcp: mass None -> 1e-05
- link openarm_right_link0: geometry collision mesh filename=package://openarm_description/meshes/arm/v10/collision/link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 scale=0.001 0.001 0.001; visual mesh filename=package://openarm_description/meshes/arm/v10/visual_right/l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 scale=0.001 0.001 0.001
- link openarm_right_link1: geometry collision mesh filename=package://openarm_description/meshes/arm/v10/collision/link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 scale=0.001 0.001 0.001; visual mesh filename=package://openarm_description/meshes/arm/v10/visual_right/l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 scale=0.001 0.001 0.001
- link openarm_right_link2: geometry collision mesh filename=package://openarm_description/meshes/arm/v10/collision/link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 scale=0.001 0.001 0.001; visual mesh filename=package://openarm_description/meshes/arm/v10/visual_right/l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 scale=0.001 0.001 0.001
- link openarm_right_link3: geometry collision mesh filename=package://openarm_description/meshes/arm/v10/collision/link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 scale=0.001 0.001 0.001; visual mesh filename=package://openarm_description/meshes/arm/v10/visual_right/l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 scale=0.001 0.001 0.001
- link openarm_right_link4: geometry collision mesh filename=package://openarm_description/meshes/arm/v10/collision/link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 scale=0.001 0.001 0.001; visual mesh filename=package://openarm_description/meshes/arm/v10/visual_right/l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 scale=0.001 0.001 0.001
- link openarm_right_link5: geometry collision mesh filename=package://openarm_description/meshes/arm/v10/collision/link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 scale=0.001 0.001 0.001; visual mesh filename=package://openarm_description/meshes/arm/v10/visual_right/l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 scale=0.001 0.001 0.001
- link openarm_right_link6: geometry collision mesh filename=package://openarm_description/meshes/arm/v10/collision/link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 scale=0.001 0.001 0.001; visual mesh filename=package://openarm_description/meshes/arm/v10/visual_right/l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 scale=0.001 0.001 0.001
- link openarm_right_link7: geometry collision mesh filename=package://openarm_description/meshes/arm/v10/collision/link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 scale=0.001 0.001 0.001; visual mesh filename=package://openarm_description/meshes/arm/v10/visual_right/l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 scale=0.001 0.001 0.001
Joints:
- joint openarm_right_joint4: origin xyz=-0.0 0.0315 0.15375 rpy=0 0 0 -> xyz=-0.0 -0.0315 0.15375 rpy=0 0 0
- joint openarm_right_joint5: origin xyz=0.0 -0.0315 0.0955 rpy=0 0 0 -> xyz=0.0 0.0315 0.0955 rpy=0 0 0
